Commit message: Added Collision and inertia

File: Assignment_3_and_4/src/cat_description/urdf/cat.urdf (robot description, URDF)
Before this commit: robot cat, 1 links, 0 joints
Links:
- removed link cat_body
- added link base_link, mass 10; collision cylinder length=0.5 radius=0.15; visual cylinder length=0.5 radius=0.15
- added link head, mass 10; collision sphere radius=0.15; visual sphere radius=0.15
- added link leg_LB, mass 10; collision cylinder length=0.25 radius=0.05; visual cylinder length=0.25 radius=0.05
- added link leg_LB_wheel, mass 10; collision cylinder length=0.06 radius=0.02; visual cylinder length=0.06 radius=0.02
- added link leg_LF, mass 10; collision cylinder length=0.25 radius=0.05; visual cylinder length=0.25 radius=0.05
- added link leg_LF_wheel, mass 10; collision cylinder length=0.06 radius=0.02; visual cylinder length=0.06 radius=0.02
- added link leg_RB, mass 10; collision cylinder length=0.25 radius=0.05; visual cylinder length=0.25 radius=0.05
- added link leg_RB_wheel, mass 10; collision cylinder length=0.06 radius=0.02; visual cylinder length=0.06 radius=0.02
- added link leg_RF, mass 10; collision cylinder length=0.25 radius=0.05; visual cylinder length=0.25 radius=0.05
- added link leg_RF_wheel, mass 10; collision cylinder length=0.06 radius=0.02; visual cylinder length=0.06 radius=0.02
Joints:
- added joint base_head: type fixed, parent base_link, child head, origin xyz=0.35 0 0.45 rpy=0 0 0
- added joint base_leg_LB: type fixed, parent base_link, child leg_LB, origin xyz=-0.2 0.075 0.125 rpy=0 0 0
- added joint base_leg_LF: type fixed, parent base_link, child leg_LF, origin xyz=0.2 0.075 0.125 rpy=0 0 0
- added joint base_leg_RB: type fixed, parent base_link, child leg_RB, origin xyz=-0.2 -0.075 0.125 rpy=0 0 0
- added joint base_leg_RF: type fixed, parent base_link, child leg_RF, origin xyz=0.2 -0.075 0.125 rpy=0 0 0
- added joint leg_LB_wheel_link: type continuous, parent leg_LB, child leg_LB_wheel, origin xyz=0 0 -0.125 rpy=1.57075 1.57075 0, axis 0 0 1, mimic joint=leg_LF_wheel_link
- added joint leg_LF_wheel_link: type continuous, parent leg_LF, child leg_LF_wheel, origin xyz=0 0 -0.125 rpy=1.57075 1.57075 0, axis 0 0 1
- added joint leg_RB_wheel_link: type continuous, parent leg_RB, child leg_RB_wheel, origin xyz=0 0 -0.125 rpy=1.57075 1.57075 0, axis 0 0 1, mimic joint=leg_RF_wheel_link
- added joint leg_RF_wheel_link: type continuous, parent leg_RF, child leg_RF_wheel, origin xyz=0 0 -0.125 rpy=1.57075 1.57075 0, axis 0 0 1
