Commit message: Removed effort and velocity limits

File: Assignment_3_and_4/src/cat_description/urdf/macros.xacro (robot description, xacro)
@@ -100,5 +100,4 @@
       <origin rpy="${PI/2} ${PI/2} 0" xyz="0 0 -${legLength/2}"/>
       <axis xyz="0 0 1"/>
-      <limit effort="100" velocity="100"/>
       <joint_properties damping="0.0" friction="0.0"/>
       <xacro:if value="${mr}">

Commit message: Axis fix

File: Assignment_3_and_4/src/cat_description/urdf/macros.xacro (robot description, xacro)
@@ -99,5 +99,5 @@
       <child link="wheel_${lr}${fb}"/>
       <origin rpy="${PI/2} ${PI/2} 0" xyz="0 0 -${legLength/2}"/>
-      <axis xyz="0 0 1"/>
+      <axis xyz="0 0 -1"/>
       <joint_properties damping="0.0" friction="0.0"/>
       <xacro:if value="${mr}">

Commit message: Laser data gathering and PointCloud implementation

File: Assignment_3_and_4/src/cat_description/urdf/macros.xacro (robot description, xacro)
@@ -137,5 +137,5 @@
       <parent link="spinner_${lr}${fb}"/>
       <child link="wheel_${lr}${fb}"/>
-      <origin rpy="${PI/2} ${PI/2} 0" xyz="0 0 -${spinnerLength/2}"/>
+      <origin rpy="${PI/2} ${PI/2} 0" xyz="0 0 0"/>
       <axis xyz="0 0 -1"/>
       <joint_properties damping="0.0" friction="0.0"/>
