Commit message: Updated .xacro files with self-suficient link templates

File: Assignment_3_and_4/src/cat_description/urdf/cat.xacro (robot description, xacro)
@@ -2,5 +2,5 @@
 <robot name="cat" xmlns:xacro="http://www.ros.org/wiki/xacro">
 	<xacro:property name="PI" value="3.1415926535897931"/>
-	<xacro:property name="bodylength" value="0.5"/>
+	<xacro:property name="bodyLength" value="0.5"/>
 	<xacro:property name="bodyRadius" value="0.15"/>
 	<xacro:property name="bodyMass" value="10"/>
@@ -19,19 +19,19 @@
 		<collision>
 			<geometry>
-				<cylinder length="${bodylength}" radius="${bodyRadius}" />
+				<cylinder length="${bodyLength}" radius="${bodyRadius}" />
 			</geometry>
-			<origin rpy="0 1.57075 0" xyz="0 0 0.3"/>
+			<origin rpy="0 ${PI/2} 0" xyz="0 0 0.3"/>
 		</collision>
 		<visual>
 			<geometry>
-				<cylinder length="${bodylength}" radius="${bodyRadius}" />
+				<cylinder length="${bodyLength}" radius="${bodyRadius}" />
 			</geometry>
-			<origin rpy="0 1.57075 0" xyz="0 0 0.3"/>
+			<origin rpy="0 ${PI/2} 0" xyz="0 0 0.3"/>
 			<material name="grey" />
 		</visual>
 		<inertial>
-			<origin rpy="0 1.57075 0" xyz="0 0 0.3"/>
+			<origin rpy="0 ${PI/2} 0" xyz="0 0 0.3"/>
 			<mass value="${bodyMass}"/>
-			<cylinder_inertia m="${bodyMass}" r="${bodyRadius}" h="${bodylength}"/>
+			<cylinder_inertia m="${bodyMass}" r="${bodyRadius}" h="${bodyLength}"/>
 		</inertial>
 	</link>
@@ -58,205 +58,11 @@
 		<origin rpy="0 0 0" xyz="0.35 0 0.45"/>
 	</joint>
-	<link name="leg_LF">
-		<visual>
-			<geometry>
-				<cylinder length="${legLength}" radius="${legRadius}" />
-			</geometry>
-			<material name="grey" />
-		</visual>
-		<collision>
-			<geometry>
-				<cylinder length="${legLength}" radius="${legRadius}" />
-			</geometry>
-		</collision>
-		<inertial>
-			<mass value="${legMass}"/>
-			<cylinder_inertia m="${legMass}" r="${legRadius}" h="${legLength}"/>
-		</inertial>
-	</link>
-	<joint name="base_leg_LF" type="fixed">
-		<parent link="base_link"/>
-		<child link="leg_LF"/>
-		<origin rpy="0 0 0" xyz="0.2 0.075 0.125"/>
-	</joint>
-	<link name="leg_LF_wheel">
-		<visual>
-			<geometry>
-				<cylinder length="${wheelLength}" radius="${wheelRadius}" />
-			</geometry>
-			<material name="grey" />
-		</visual>
-		<collision>
-			<geometry>
-				<cylinder length="${wheelLength}" radius="${wheelRadius}" />
-			</geometry>
-		</collision>
-		<inertial>
-			<mass value="${wheelMass}"/>
-			<cylinder_inertia m="${wheelMass}" r="${wheelRadius}" h="${wheelLength}"/>
-		</inertial>
-	</link>
-	<joint name="leg_LF_wheel_link" type="continuous">
-		<parent link="leg_LF"/>
-		<child link="leg_LF_wheel"/>
-		<origin rpy="1.57075 1.57075 0" xyz="0 0 -0.125"/>
-		<axis xyz="0 0 1" />
-	</joint>
-	<link name="leg_RF">
-		<visual>
-			<geometry>
-				<cylinder length="${legLength}" radius="${legRadius}" />
-			</geometry>
-			<material name="grey" />
-		</visual>
-		<collision>
-			<geometry>
-				<cylinder length="${legLength}" radius="${legRadius}" />
-			</geometry>
-		</collision>
-		<inertial>
-			<mass value="${legMass}"/>
-			<cylinder_inertia m="${legMass}" r="${legRadius}" h="${legLength}"/>
-		</inertial>
-	</link>
-	<joint name="base_leg_RF" type="fixed">
-		<parent link="base_link"/>
-		<child link="leg_RF"/>
-		<origin rpy="0 0 0" xyz="0.2 -0.075 0.125"/>
-	</joint>
-	<link name="leg_RF_wheel">
-		<visual>
-			<geometry>
-				<cylinder length="${wheelLength}" radius="${wheelRadius}" />
-			</geometry>
-			<material name="grey" />
-		</visual>
-		<collision>
-			<geometry>
-				<cylinder length="${wheelLength}" radius="${wheelRadius}" />
-			</geometry>
-		</collision>
-		<inertial>
-			<mass value="${wheelMass}"/>
-			<cylinder_inertia m="${wheelMass}" r="${wheelRadius}" h="${wheelLength}"/>
-		</inertial>
-	</link>
-	<joint name="leg_RF_wheel_link" type="continuous">
-		<parent link="leg_RF"/>
-		<child link="leg_RF_wheel"/>
-		<origin rpy="1.57075 1.57075 0" xyz="0 0 -0.125"/>
-		<axis xyz="0 0 1" />
-	</joint>
-	<link name="leg_LB">
-		<visual>
-			<geometry>
-				<cylinder length="${legLength}" radius="${legRadius}" />
-			</geometry>
-			<material name="grey" />
-		</visual>
-		<collision>
-			<geometry>
-				<cylinder length="${legLength}" radius="${legRadius}" />
-			</geometry>
-		</collision>
-		<inertial>
-			<mass value="${legMass}"/>
-			<cylinder_inertia m="${legMass}" r="${legRadius}" h="${legLength}"/>
-		</inertial>
-	</link>
-	<joint name="base_leg_LB" type="fixed">
-		<parent link="base_link"/>
-		<child link="leg_LB"/>
-		<origin rpy="0 0 0" xyz="-0.2 0.075 0.125"/>
-	</joint>
-	<link name="leg_LB_wheel">
-		<visual>
-			<geometry>
-				<cylinder length="${wheelLength}" radius="${wheelRadius}" />
-			</geometry>
-			<material name="grey" />
-		</visual>
-		<collision>
-			<geometry>
-				<cylinder length="${wheelLength}" radius="${wheelRadius}" />
-			</geometry>
-		</collision>
-		<inertial>
-			<mass value="${wheelMass}"/>
-			<cylinder_inertia m="${wheelMass}" r="${wheelRadius}" h="${wheelLength}"/>
-		</inertial>
-	</link>
-	<joint name="leg_LB_wheel_link" type="continuous">
-		<parent link="leg_LB"/>
-		<child link="leg_LB_wheel"/>
-		<origin rpy="1.57075 1.57075 0" xyz="0 0 -0.125"/>
-		<axis xyz="0 0 1" />
-		<mimic joint="leg_LF_wheel_link"/>
-	</joint>
-	<link name="leg_RB">
-		<visual>
-			<geometry>
-				<cylinder length="${legLength}" radius="${legRadius}" />
-			</geometry>
-			<material name="grey" />
-		</visual>
-		<collision>
-			<geometry>
-				<cylinder length="${legLength}" radius="${legRadius}" />
-			</geometry>
-		</collision>
-		<inertial>
-			<mass value="${legMass}"/>
-			<cylinder_inertia m="${legMass}" r="${legRadius}" h="${legLength}"/>
-		</inertial>
-	</link>
-	<joint name="base_leg_RB" type="fixed">
-		<parent link="base_link"/>
-		<child link="leg_RB"/>
-		<origin rpy="0 0 0" xyz="-0.2 -0.075 0.125"/>
-	</joint>
-	<link name="leg_RB_wheel">
-		<visual>
-			<geometry>
-				<cylinder length="${wheelLength}" radius="${wheelRadius}" />
-			</geometry>
-			<material name="grey" />
-		</visual>
-		<collision>
-			<geometry>
-				<cylinder length="${wheelLength}" radius="${wheelRadius}" />
-			</geometry>
-		</collision>
-		<inertial>
-			<mass value="${wheelMass}"/>
-			<cylinder_inertia m="${wheelMass}" r="${wheelRadius}" h="${wheelLength}"/>
-		</inertial>
-	</link>
-	<joint name="leg_RB_wheel_link" type="continuous">
-		<parent link="leg_RB"/>
-		<child link="leg_RB_wheel"/>
-		<origin rpy="1.57075 1.57075 0" xyz="0 0 -0.125"/>
-		<axis xyz="0 0 1" />
-		<mimic joint="leg_RF_wheel_link"/>
-	</joint>
-	<transmission name="left_trans">
-		<type>transmission_interface/SimpleTransmission</type>
-		<joint name="leg_LF_wheel_link">
-			<hardwareInterface>hardware_interface/EffortJointInterface</hardwareInterface>
-		</joint>
-		<actuator name="LT">
-			<hardwareInterface>hardware_interface/EffortJointInterface</hardwareInterface>
-			<mechanicalReduction>1</mechanicalReduction>
-		</actuator>
-	</transmission>
-	<transmission name="right_trans">
-		<type>transmission_interface/SimpleTransmission</type>
-		<joint name="leg_RF_wheel_link">
-			<hardwareInterface>hardware_interface/EffortJointInterface</hardwareInterface>
-		</joint>
-		<actuator name="RT">
-			<hardwareInterface>hardware_interface/EffortJointInterface</hardwareInterface>
-			<mechanicalReduction>1</mechanicalReduction>
-		</actuator>
-	</transmission>
+	<leg lr="L" fb="F" tY="1" tX="1" />
+	<leg lr="R" fb="F" tY="-1" tX="1" />
+	<leg lr="L" fb="B" tY="1" tX="-1" />
+	<leg lr="R" fb="B" tY="-1" tX="-1" />
+	<wheel lr="L" fb="F" mr="0" mlr="" mfb=""/>
+	<wheel lr="R" fb="F" mr="0" mlr="" mfb=""/>
+	<wheel lr="L" fb="B" mr="1" mlr="L" mfb="F"/>
+	<wheel lr="R" fb="B" mr="1" mlr="R" mfb="F"/>
 </robot>

File: Assignment_3_and_4/src/cat_description/urdf/macros.xacro (robot description, xacro)
@@ -1,4 +1,9 @@
 <?xml version="1.0"?>
 <robot xmlns:xacro="http://www.ros.org/wiki/xacro">
+  <!--
+    m = mass
+    r = radius
+    h = height
+  -->
   <xacro:macro name="cylinder_inertia" params="m r h">
     <inertia  ixx="${m*(3*r*r+h*h)/12}" ixy = "0" ixz = "0"
@@ -7,4 +12,10 @@
     />
   </xacro:macro>
+  <!--
+    m = mass
+    x = x value
+    y = y value
+    z = z value
+  -->
   <xacro:macro name="box_inertia" params="m x y z">
     <inertia  ixx="${m*(y*y+z*z)/12}" ixy = "0" ixz = "0"
@@ -13,4 +24,8 @@
     />
   </xacro:macro>
+  <!--
+    m = mass
+    r = radius
+  -->
   <xacro:macro name="sphere_inertia" params="m r">
     <inertia  ixx="${2*m*r*r/5}" ixy = "0" ixz = "0"
@@ -19,3 +34,86 @@
     />
   </xacro:macro>
+  <!--
+    lr = left/right ("L" | "R")
+    fb = front/back ("F" | "B")
+    tY = translation in Y ("1" | "-1")
+    tX = translation in X ("1" | "-1")
+  -->
+  <xacro:macro name="leg" params="lr fb tY tX">
+    <link name="leg_${lr}${fb}">
+      <collision>
+        <geometry>
+          <cylinder length="${legLength}" radius="${legRadius}" />
+        </geometry>
+      </collision>
+      <visual>
+        <geometry>
+          <cylinder length="${legLength}" radius="${legRadius}" />
+        </geometry>
+        <material name="grey" />
+      </visual>
+      <inertial>
+        <mass value="${legMass}"/>
+        <cylinder_inertia m="${legMass}" r="${legRadius}" h="${legLength}"/>
+      </inertial>
+    </link>
+    <gazebo reference="leg_${lr}${fb}">
+      <material>Gazebo/Grey</material>
+    </gazebo>
+    <joint name="body_leg_${lr}${fb}_joint" type="fixed">
+      <parent link="base_link"/>
+      <child link="leg_${lr}${fb}"/>
+      <origin rpy="0 0 0" xyz="${tX*2*bodyLength/5} ${tY*bodyRadius/2} ${legLength/2}"/>
+    </joint>
+  </xacro:macro>
+  <!--
+    lr = left/right ("L" | " R")
+    fb = front/back ("F" | "B")
+    mr = mirror (Boolean | "")
+    mlr = mirror left/right ("L" | "R")
+    mfb = mirror front/back ("F" | "B")
+  -->
+  <xacro:macro name="wheel" params="lr fb mr mlr mfb">
+    <link name="wheel_${lr}${fb}">
+      <collision>
+        <geometry>
+          <cylinder length="${wheelLength}" radius="${wheelRadius}" />
+        </geometry>
+      </collision>
+      <visual>
+        <geometry>
+          <cylinder length="${wheelLength}" radius="${wheelRadius}" />
+        </geometry>
+        <material name="black" />
+      </visual>
+      <inertial>
+        <mass value="${wheelMass}"/>
+        <cylinder_inertia m="${wheelMass}" r="${wheelRadius}" h="${wheelLength}"/>
+      </inertial>
+    </link>
+    <gazebo reference="wheel_${lr}${fb}">
+      <material>Gazebo/Black</material>
+    </gazebo>
+    <joint name="leg_wheel_${lr}${fb}_joint" type="continuous">
+      <parent link="leg_${lr}${fb}"/>
+      <child link="wheel_${lr}${fb}"/>
+      <origin rpy="${PI/2} ${PI/2} 0" xyz="0 0 -${legLength/2}"/>
+      <axis xyz="0 0 1"/>
+      <limit effort="100" velocity="100"/>
+      <joint_properties damping="0.0" friction="0.0"/>
+      <xacro:if value="${mr}">
+        <mimic joint="leg_wheel_${mlr}${mfb}_joint"/>
+      </xacro:if>
+    </joint>
+    <transmission name="trans_${lr}${fb}">
+      <type>transmission_interface/SimpleTransmission</type>
+      <joint name="leg_wheel_${lr}${fb}_joint">
+        <hardwareInterface>hardware_interface/EffortJointInterface</hardwareInterface>
+      </joint>
+      <actuator name="motor_${lr}${fb}">
+        <hardwareInterface>hardware_interface/EffortJointInterface</hardwareInterface>
+        <mechanicalReduction>1</mechanicalReduction>
+      </actuator>
+    </transmission>
+  </xacro:macro>
 </robot>

Commit message: Some worlds

File: Assignment_3_and_4/src/cat_description/urdf/cat.xacro (robot description, xacro)
@@ -66,3 +66,29 @@
 	<wheel lr="L" fb="B" mr="1" mlr="L" mfb="F"/>
 	<wheel lr="R" fb="B" mr="1" mlr="R" mfb="F"/>
+	<joint name="hokuyo_joint" type="fixed">
+		<axis xyz="0 0 0" />
+		<origin xyz="0 0 0" rpy="0 0 0"/>
+		<parent link="head"/>
+		<child link="hokuyo_link"/>
+  	</joint>
+	<!-- Hokuyo Laser -->
+	<link name="hokuyo_link">
+		<collision>
+		<origin xyz="0 0 0" rpy="0 0 0"/>
+		<geometry>
+		<box size="0.1 0.1 0.1"/>
+		</geometry>
+		</collision>
+		<visual>
+		<origin xyz="0 0 0" rpy="0 0 0"/>
+		<geometry>
+			<box size="0.1 0.1 0.1"/>
+		</geometry>
+		</visual>
+		<inertial>
+		<mass value="1e-5" />
+		<origin xyz="0 0 0" rpy="0 0 0"/>
+		<inertia ixx="1e-6" ixy="0" ixz="0" iyy="1e-6" iyz="0" izz="1e-6" />
+		</inertial>
+	</link>
 </robot>

Commit message: The wheels on the cat go round and round

File: Assignment_3_and_4/src/cat_description/urdf/cat.xacro (robot description, xacro)
@@ -4,5 +4,5 @@
 	<xacro:property name="bodyLength" value="0.5"/>
 	<xacro:property name="bodyRadius" value="0.15"/>
-	<xacro:property name="bodyMass" value="10"/>
+	<xacro:property name="bodyMass" value="100"/>
 	<xacro:property name="headRadius" value="0.15"/>
 	<xacro:property name="headMass" value="10"/>
@@ -10,4 +10,7 @@
 	<xacro:property name="legRadius" value="0.05"/>
 	<xacro:property name="legMass" value="10"/>
+	<xacro:property name="spinnerLength" value="0.01"/>
+	<xacro:property name="spinnerRadius" value="0.04"/>
+	<xacro:property name="spinnerMass" value="1"/>
 	<xacro:property name="wheelLength" value="0.06"/>
 	<xacro:property name="wheelRadius" value="0.02"/>
@@ -62,8 +65,10 @@
 	<leg lr="L" fb="B" tY="1" tX="-1" />
 	<leg lr="R" fb="B" tY="-1" tX="-1" />
-	<wheel lr="L" fb="F" mr="0" mlr="" mfb=""/>
-	<wheel lr="R" fb="F" mr="0" mlr="" mfb=""/>
-	<wheel lr="L" fb="B" mr="1" mlr="L" mfb="F"/>
-	<wheel lr="R" fb="B" mr="1" mlr="R" mfb="F"/>
+	<spinner lr="L" fb="F" tY="1" tX="1" />
+	<spinner lr="R" fb="F" tY="1" tX="1" />
+	<wheel lr="L" fb="F"/>
+	<wheel lr="R" fb="F"/>
+	<wheelB lr="L" fb="B"/>
+	<wheelB lr="R" fb="B"/>
 	<joint name="hokuyo_joint" type="fixed">
 		<axis xyz="0 0 0" />

File: Assignment_3_and_4/src/cat_description/urdf/macros.xacro (robot description, xacro)
@@ -67,4 +67,43 @@
     </joint>
   </xacro:macro>
+  <xacro:macro name="spinner" params="lr fb tY tX">
+    <link name="spinner_${lr}${fb}">
+      <collision>
+        <geometry>
+          <cylinder length="${spinnerLength}" radius="${spinnerRadius}" />
+        </geometry>
+      </collision>
+      <visual>
+        <geometry>
+          <cylinder length="${spinnerLength}" radius="${spinnerRadius}" />
+        </geometry>
+        <material name="grey" />
+      </visual>
+      <inertial>
+        <mass value="${spinnerMass}"/>
+        <cylinder_inertia m="${spinnerMass}" r="${spinnerRadius}" h="${spinnerLength}"/>
+      </inertial>
+    </link>
+    <gazebo reference="leg_${lr}${fb}">
+      <material>Gazebo/Grey</material>
+    </gazebo>
+    <joint name="leg_${lr}${fb}_spinner_joint" type="revolute">
+      <parent link="leg_${lr}${fb}"/>
+      <child link="spinner_${lr}${fb}"/>
+      <limit lower="-0.7" upper="0.7" effort="1000" velocity="1000"/>
+      <origin rpy="0 0 0" xyz="0 0 -${legLength/2}"/>
+      <axis xyz="0 0 1"/>
+    </joint>
+    <transmission name="trans_spin_${lr}${fb}">
+      <type>transmission_interface/SimpleTransmission</type>
+      <joint name="leg_${lr}${fb}_spinner_joint">
+        <hardwareInterface>hardware_interface/EffortJointInterface</hardwareInterface>
+      </joint>
+      <actuator name="motor_spin_${lr}${fb}">
+        <hardwareInterface>hardware_interface/EffortJointInterface</hardwareInterface>
+        <mechanicalReduction>1</mechanicalReduction>
+      </actuator>
+    </transmission>
+  </xacro:macro>
   <!--
     lr = left/right ("L" | " R")
@@ -74,5 +113,34 @@
     mfb = mirror front/back ("F" | "B")
   -->
-  <xacro:macro name="wheel" params="lr fb mr mlr mfb">
+  <xacro:macro name="wheel" params="lr fb">
+    <link name="wheel_${lr}${fb}">
+      <collision>
+        <geometry>
+          <cylinder length="${wheelLength}" radius="${wheelRadius}" />
+        </geometry>
+      </collision>
+      <visual>
+        <geometry>
+          <cylinder length="${wheelLength}" radius="${wheelRadius}" />
+        </geometry>
+        <material name="black" />
+      </visual>
+      <inertial>
+        <mass value="${wheelMass}"/>
+        <cylinder_inertia m="${wheelMass}" r="${wheelRadius}" h="${wheelLength}"/>
+      </inertial>
+    </link>
+    <gazebo reference="wheel_${lr}${fb}">
+      <material>Gazebo/Black</material>
+    </gazebo>
+    <joint name="leg_wheel_${lr}${fb}_joint" type="continuous">
+      <parent link="spinner_${lr}${fb}"/>
+      <child link="wheel_${lr}${fb}"/>
+      <origin rpy="${PI/2} ${PI/2} 0" xyz="0 0 -${spinnerLength/2}"/>
+      <axis xyz="0 0 -1"/>
+      <joint_properties damping="0.0" friction="0.0"/>
+    </joint>
+  </xacro:macro>
+  <xacro:macro name="wheelB" params="lr fb">
     <link name="wheel_${lr}${fb}">
       <collision>
@@ -101,7 +169,4 @@
       <axis xyz="0 0 -1"/>
       <joint_properties damping="0.0" friction="0.0"/>
-      <xacro:if value="${mr}">
-        <mimic joint="leg_wheel_${mlr}${mfb}_joint"/>
-      </xacro:if>
     </joint>
     <transmission name="trans_${lr}${fb}">

Commit message: Ackermann steering

File: Assignment_3_and_4/src/cat_description/urdf/cat.xacro (robot description, xacro)
@@ -65,6 +65,6 @@
 	<leg lr="L" fb="B" tY="1" tX="-1" />
 	<leg lr="R" fb="B" tY="-1" tX="-1" />
-	<spinner lr="L" fb="F" tY="1" tX="1" />
-	<spinner lr="R" fb="F" tY="1" tX="1" />
+	<spinnerL R="0.5"/>
+	<spinnerR R="0.5"/>
 	<wheel lr="L" fb="F"/>
 	<wheel lr="R" fb="F"/>

File: Assignment_3_and_4/src/cat_description/urdf/macros.xacro (robot description, xacro)
@@ -67,6 +67,6 @@
     </joint>
   </xacro:macro>
-  <xacro:macro name="spinner" params="lr fb tY tX">
-    <link name="spinner_${lr}${fb}">
+  <xacro:macro name="spinnerL" params="R">
+    <link name="spinner_LF">
       <collision>
         <geometry>
@@ -85,20 +85,59 @@
       </inertial>
     </link>
-    <gazebo reference="leg_${lr}${fb}">
+    <gazebo reference="leg_LF">
       <material>Gazebo/Grey</material>
     </gazebo>
-    <joint name="leg_${lr}${fb}_spinner_joint" type="revolute">
-      <parent link="leg_${lr}${fb}"/>
-      <child link="spinner_${lr}${fb}"/>
-      <limit lower="-0.7" upper="0.7" effort="1000" velocity="1000"/>
+    <joint name="leg_LF_spinner_joint" type="revolute">
+      <parent link="leg_LF"/>
+      <child link="spinner_LF"/>
+      <limit lower="-${atan((4*bodyLength/5)/(R + bodyRadius/2))}" upper="${atan((4*bodyLength/5)/(R - bodyRadius/2))}" effort="1000" velocity="1000"/>
       <origin rpy="0 0 0" xyz="0 0 -${legLength/2}"/>
       <axis xyz="0 0 1"/>
     </joint>
-    <transmission name="trans_spin_${lr}${fb}">
+    <transmission name="trans_spin_LF">
       <type>transmission_interface/SimpleTransmission</type>
-      <joint name="leg_${lr}${fb}_spinner_joint">
+      <joint name="leg_LF_spinner_joint">
         <hardwareInterface>hardware_interface/EffortJointInterface</hardwareInterface>
       </joint>
-      <actuator name="motor_spin_${lr}${fb}">
+      <actuator name="motor_spin_LF">
+        <hardwareInterface>hardware_interface/EffortJointInterface</hardwareInterface>
+        <mechanicalReduction>1</mechanicalReduction>
+      </actuator>
+    </transmission>
+  </xacro:macro>
+  <xacro:macro name="spinnerR" params="R">
+    <link name="spinner_RF">
+      <collision>
+        <geometry>
+          <cylinder length="${spinnerLength}" radius="${spinnerRadius}" />
+        </geometry>
+      </collision>
+      <visual>
+        <geometry>
+          <cylinder length="${spinnerLength}" radius="${spinnerRadius}" />
+        </geometry>
+        <material name="grey" />
+      </visual>
+      <inertial>
+        <mass value="${spinnerMass}"/>
+        <cylinder_inertia m="${spinnerMass}" r="${spinnerRadius}" h="${spinnerLength}"/>
+      </inertial>
+    </link>
+    <gazebo reference="leg_RF">
+      <material>Gazebo/Grey</material>
+    </gazebo>
+    <joint name="leg_RF_spinner_joint" type="revolute">
+      <parent link="leg_RF"/>
+      <child link="spinner_RF"/>
+      <limit lower="-${atan((4*bodyLength/5)/(R - bodyRadius/2))}" upper="${atan((4*bodyLength/5)/(R + bodyRadius/2))}" effort="1000" velocity="1000"/>
+      <origin rpy="0 0 0" xyz="0 0 -${legLength/2}"/>
+      <axis xyz="0 0 1"/>
+    </joint>
+    <transmission name="trans_spin_RF">
+      <type>transmission_interface/SimpleTransmission</type>
+      <joint name="leg_RF_spinner_joint">
+        <hardwareInterface>hardware_interface/EffortJointInterface</hardwareInterface>
+      </joint>
+      <actuator name="motor_spin_RF">
         <hardwareInterface>hardware_interface/EffortJointInterface</hardwareInterface>
         <mechanicalReduction>1</mechanicalReduction>
